File: KiCAD/smartyreader_v2_lora/smartyreader_ng_lora.kicad_pcb (KiCad board)
At the start: 2 copper layers, 57.1 x 30.5 mm, 21 parts, among them J1 Smartmeter RJ12, J2 I2C_Header, J3 W5100_2x5, J4 3.3V_H1, J5 5V_H1, J6 Conn_Coaxial, J7 ANT, U1 RFM95W

Commit message: corrected links
Parts:
- removed AD1 (x2): C1, weigu:WPin_3mm
- removed JP1: RESET, weigu:W0805
- removed JP2: IRQ_DIO1, weigu:W0805
- removed REF**: OSHW-Logo2_7.3x6mm_SilkScreen, Symbol:OSHW-Logo2_7.3x6mm_SilkScreen
- removed REF**: OSHW-Logo2_9.8x8mm_SilkScreen, Symbol:OSHW-Logo2_9.8x8mm_SilkScreen
- added D1: 1N4148, weigu:W0805, B.Cu at (153.7, 111.7)
- added D2: 1N4148, weigu:W0805, B.Cu at (156.0, 111.8)
- added H1: WMHole, weigu:WPin_3mm, F.Cu at (104.1, 108.0)
- added H2: WMHole, weigu:WPin_3mm, F.Cu at (153.7, 130.8)
- added LOGO?1: Open_Hardware_Logo, Symbol:OSHW-Logo_5.7x6mm_SilkScreen, B.Cu at (123.4, 116.1)
- added LOGO?2: Open_Hardware_Logo, Symbol:OSHW-Logo_5.7x6mm_SilkScreen, F.Cu at (131.1, 116.5)
Connections:
- J3 pad 7: Net-(J3-Pad7) -> Net-(D1-Pad2)
- U1 pad 14: Net-(J3-Pad7) -> Net-(D1-Pad1)
- U1 pad 6: Net-(JP1-Pad2) -> Net-(U1-Pad6)
- W1 pad 15: Net-(J3-Pad7) -> Net-(D1-Pad2)
- W1 pad 3: Net-(JP1-Pad1) -> (no net)
- W1 pad 4: Net-(JP2-Pad1) -> (no net)
- W1 pad 9: (no net) -> Net-(U1-Pad6)
Routing:
- net Net-(J3-Pad7): track 59.3 -> 0.00 mm, vias 3 -> 0
- net Net-(D1-Pad2): track 0.00 -> 36.3 mm, vias 0 -> 1
- net Net-(JP1-Pad2): track 34.4 -> 0.00 mm
- net Net-(D1-Pad1): track 0.00 -> 18.6 mm
- net Net-(D2-Pad1): track 6.16 -> 21.3 mm
- net Net-(JP2-Pad1): track 6.94 -> 0.00 mm
- net Net-(U1-Pad6): track 0.00 -> 4.91 mm
- net ~: track 173.9 -> 169.4 mm
- net Net-(JP1-Pad1): track 2.92 -> 0.00 mm
Other:
- board text added: "SmartyReader v 2.1 05/21 by weigu.lu"
- board text added: "smartyreader v. 2.1 05/21 by weigu.lu"
- board text removed: "SmartyReader v 2.0 02/21 by weigu.lu"
- board text removed: "smartyreader v. 2.0 02/21 by weigu.lu"
